Commit message: Changes colors of wheels

File: project2/my_robot/urdf/my_robot.xacro (robot description, xacro)
@@ -181,8 +181,8 @@
   </joint>
 <gazebo reference="left_wheel">
-    <material>Gazebo/Green</material>
+    <material>Gazebo/Black</material>
 </gazebo>
 <gazebo reference="right_wheel">
-    <material>Gazebo/Green</material>
+    <material>Gazebo/Black</material>
 </gazebo>
 <gazebo reference="camera">
